File: TNU_PIC18F_Microcontroller_Board.kicad_sch (KiCad schematic)
At the start: 4 parts, among them J1 USB_B_Micro, U1 FT231XS

Commit message: Removed accidental 3.3V to USB D+ short circuit
Parts:
- added C1: 100uF, Capacitor_SMD:C_0805_2012Metric, symbol Device:C
- added C2: 22uF, Capacitor_SMD:C_0805_2012Metric, symbol Device:C
- added U2: LD1117S33TR_SOT223, Package_TO_SOT_SMD:SOT-223-3_TabPin2, symbol Regulator_Linear:LD1117S33TR_SOT223
Connections:
- net GND: now also C1.2, C2.2, U2.1 (GND)
- new net: C2.1, U2.2 (VO)
- new net: C1.1, U2.3 (VI)

Commit message: COMPLETED: Full Cadence-to-KiCad translation with complete ICSP programming header wiring
Parts:
- added J2: Conn_01x06_Pin, Connector_PinHeader_2.54mm:PinHeader_1x06_P2.54mm_Vertical, symbol Connector:Conn_01x06_Pin
- added U3: PIC18F4520-xP, Package_DIP:DIP-40_W15.24mm, symbol MCU_Microchip_PIC18:PIC18F4520-xP
Connections:
- net GND: now also U3.12 (VSS), U3.31 (VSS)
- net +3.3V: now reaches C2.1, U2.2 (VO)
- net +3.3V: now also U3.11 (VDD), U3.32 (VDD)
- new net: J2.1 (Pin_1), U3.1 (RE3/~{MCLR})
- new net: J2.5 (Pin_5), U3.39 (RB6)
- new net: J2.4 (Pin_4), U3.40 (RB7)

Commit message: SUBMISSION: Fully complete Cadence to KiCad schematic translation with all interface and ICSP wiring
Connections:
- net +3.3V: now also J2.2 (Pin_2)
- net GND: now also J2.3 (Pin_3)
Changed lines of the file:
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@@
+	(wire
+		(pts
+			(xy 247.65 86.36) (xy 247.65 156.21)
+		)
+		(stroke
+			(width 0)
+			(type default)
+		)
+	)
 	(wire
 		(pts
@@
 	(wire
 		(pts
+			(xy 243.84 83.82) (xy 240.03 83.82)
+		)
+		(stroke
+			(width 0)
+			(type default)
+		)
+	)
+	(wire
+		(pts
 			(xy 189.23 149.86) (xy 189.23 133.35)
 		)
@@
 	(wire
 		(pts
+			(xy 240.03 86.36) (xy 247.65 86.36)
+		)
+		(stroke
+			(width 0)
+			(type default)
+		)
+	)
+	(wire
+		(pts
 			(xy 83.82 120.65) (xy 91.44 120.65)
 		)
@@
 			(width 0)
 			(type default)
+		)
+	)
+	(global_label "+3.3V"
+		(shape input)
+		(at 243.84 83.82 0)
+		(fields_autoplaced yes)
+		(effects
+			(font
+				(size 1.27 1.27)
+			)
+			(justify left)
+		)
+		(property "Intersheetrefs" "${INTERSHEET_REFS}"
+			(at 251.8558 83.82 0)
+			(hide yes)
+			(show_name no)
+			(do_not_autoplace no)
+			(effects
+				(font
+					(size 1.27 1.27)
+				)
+				(justify left)
+			)
 		)
 	)
@@
 					(unit 1)
 				)
+			)
+		)
+	)
+	(symbol
+		(lib_id "power:GND")
+		(at 247.65 156.21 0)
+		(unit 1)
+		(body_style 1)
+		(exclude_from_sim no)
+		(in_bom yes)
+		(on_board yes)
+		(in_pos_files yes)
+		(dnp no)
+		(fields_autoplaced yes)
+		(property "Reference" "#PWR04"
+			(at 247.65 162.56 0)
+			(hide yes)
+			(show_name no)
+			(do_not_autoplace no)
+			(effects
+				(font
+					(size 1.27 1.27)
+				)
+			)
+		)
+		(property "Value" "GND"
+			(at 247.65 161.29 0)
+			(show_name no)
+			(do_not_autoplace no)
+			(effects
+				(font
+					(size 1.27 1.27)
+				)
+			)
+		)
+		(property "Footprint" ""
+			(at 247.65 156.21 0)
+			(hide yes)
+			(show_name no)
+			(do_not_autoplace no)
+			(effects
+				(font
+					(size 1.27 1.27)
+				)
+			)
+		)
+		(property "Datasheet" ""
+			(at 247.65 156.21 0)
+			(hide yes)
+			(show_name no)
+			(do_not_autoplace no)
+			(effects
+				(font
+					(size 1.27 1.27)
+				)
+			)
+		)
+		(property "Description" "Power symbol creates a global label with name \"GND\" , ground"
+			(at 247.65 156.21 0)
+			(hide yes)
+			(show_name no)
+			(do_not_autoplace no)
+			(effects
+				(font
+					(size 1.27 1.27)
+				)
+			)
+		)
+		(pin "1"
+		)
+		(instances
+			(project "TNU_PIC18F_Microcontroller_Board"
+				(path "/15e8ab22-65cb-40fd-9dcb-5e4dfc708a47"
+					(reference "#PWR04")
+					(unit 1)
+				)

Commit message: FINAL SUBMISSION: Schematic finalized with correct PIC18F47Q84 numbering and clean GND net tagging
Parts:
- U3: value PIC18F4520-xP -> PIC18F47Q84
Connections:
- net GND: now also J1.5 (GND)
Changed lines of the file:
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@@
+	(wire
+		(pts
+			(xy 105.41 92.71) (xy 105.41 90.17)
+		)
+		(stroke
+			(width 0)
+			(type default)
+		)
+	)
 	(wire
 		(pts
@@
 			(width 0)
 			(type default)
+		)
+	)
+	(label "GND"
+		(at 105.41 92.71 0)
+		(effects
+			(font
+				(size 1.27 1.27)
+			)
+			(justify left bottom)
 		)
 	)
@@
 			)
 		)
-		(property "Value" "PIC18F4520-xP"
+		(property "Value" "PIC18F47Q84"
 			(at 207.8833 77.47 0)
 			(show_name no)
