File: microcontroller.kicad_sch (KiCad schematic)
At the start: 85 parts, among them J1 SCREWTERM, J2 JUMPER2, J3 JUMPER3, J4 JUMPER2, J5 PICKIT3, P1 TP, P11 TP, P12 TP, P13 TP, P14 TP, P15 TP, P16 TP, P17 TP, P18 TP, P19 TP, P2 TP, P3 TP, P4 TP, P5 TP, P6 TP, SW1 SW KEY-SPST, U2 LD1117-3.3/SOT223, U3 PIC18F47Q84, U4 636L3C016M00000

Commit message: Fix CLK net: U4 OUT to U3 pin 13
Move CLK label and wire stub from U3 pin 14 (RA6/OSC2/CLKO) to pin 13
(OSC1/CLKIN); add no-connect flag on pin 14 (unused per Cadence PDF).
ERC 26 -> 23. DRC unchanged (84 + 152 unconnected); 2 expected parity
warnings on U3 pads 13/14 until the PCB is updated from the schematic.

Co-Authored-By: Claude Opus 5.5 <noreply@anthropic.com>
Connections:
- net CLK: now also U3.13 (OSC1/CLKIN); no longer U3.14 (RA6/OSC2/CLKO)
- no-connect marks 1 -> 2
Changed lines of the file:
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@@
+	)
+	(no_connect
+		(at 125.73 78.74)
 	)
 	(no_connect
@@
 	(wire
 		(pts
-			(xy 121.92 78.74) (xy 125.73 78.74)
+			(xy 121.92 83.82) (xy 125.73 83.82)
 		)
 		(stroke
@@
 	)
 	(label "CLK"
-		(at 121.92 78.74 180)
+		(at 121.92 83.82 180)
 		(effects
 			(font

Commit message: Wire SCL/SDA/RB3 labels to U3 RC3/RC4/RB3
Add local labels on U3 pin 18 (RC3, SCL), pin 23 (RC4, SDA) and
pin 36 (RB3), per the Cadence PDF, so R11, R12 and R8/D3 reach the MCU.
ERC 23 -> 20. DRC 84 + 152 unconnected; parity 2 -> 8 (net renames on
U3 pads 18/23/36 and TP31/TP32/TP8, cleared by Update PCB from Schematic).

Co-Authored-By: Claude Opus 5.5 <noreply@anthropic.com>
Connections:
- net RB3: now also TP8.1, U3.36 (RB3/CCP2)
- net SCL: now also TP31.1, U3.18 (SCK/SCL/RC3)
- net SDA: now also TP32.1, U3.23 (SDI/SDA/RC4)
Changed lines of the file:
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@@
+		)
+	)
+	(label "SCL"
+		(at 176.53 66.04 0)
+		(effects
+			(font
+				(size 1.27 1.27)
+			)
+			(justify left bottom)
+		)
+	)
+	(label "SDA"
+		(at 176.53 68.58 0)
+		(effects
+			(font
+				(size 1.27 1.27)
+			)
+			(justify left bottom)
+		)
+	)
+	(label "RB3"
+		(at 125.73 96.52 180)
+		(effects
+			(font
+				(size 1.27 1.27)
+			)
+			(justify right bottom)
 		)
 	)

Commit message: ERC cleanup: NC flags, PWR_FLAGs, remove stray #PWR012, usb->GND
- No-connect flags on FT231XS U1 pins 1 (DTR), 5 (RI), 7 (DSR), 8 (DCD).
- Delete floating "usb" ground symbol #PWR012.
- Change the 7 remaining "usb" (power:GNDD) grounds to power:GND; same net.
- PWR_FLAG on VCC5_USB (#FLG01), VCC (#FLG02) and the J1 input rail
  (#FLG03); two wires split at the flag points, with junctions.
- Re-enable the "footprint doesn't match footprint filters" ERC check.

ERC 20 -> 9 (8 remaining are the Step 2 USB UART issues, plus 1 new
footprint_filter warning on U4, already in the footprint fix list).
DRC unchanged: 84 + 152 unconnected + 8 known parity issues.

Co-Authored-By: Claude Opus 5.5 <noreply@anthropic.com>
Changed lines of the file:
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@@
 	(paper "A4")
 	(junction
+		(at 60.96 50.8)
+		(diameter 0)
+		(color 0 0 0 0)
+	)
+	(junction
 		(at 151.13 119.38)
 		(diameter 0)
@@
 	(wire
 		(pts
-			(xy 57.15 50.8) (xy 64.77 50.8)
+			(xy 57.15 50.8) (xy 60.96 50.8)
+		)
+		(stroke
+			(width 0)
+			(type default)
+		)
+	)
+	(wire
+		(pts
+			(xy 60.96 50.8) (xy 64.77 50.8)
 		)
 		(stroke
@@
 					(unit 1)
 				)
+			)
+		)
+	)
+	(symbol
+		(lib_id "power:PWR_FLAG")
+		(at 102.87 96.52 0)
+		(unit 1)
+		(body_style 1)
+		(exclude_from_sim no)
+		(in_bom yes)
+		(on_board yes)
+		(in_pos_files yes)
+		(dnp no)
+		(fields_autoplaced yes)
+		(property "Reference" "#FLG02"
+			(at 102.87 94.615 0)
+			(hide yes)
+			(show_name no)
+			(do_not_autoplace no)
+			(effects
+				(font
+					(size 1.27 1.27)
+				)
+			)
+		)
+		(property "Value" "PWR_FLAG"
+			(at 102.87 92.71 0)
+			(show_name no)
+			(do_not_autoplace no)
+			(effects
+				(font
+					(size 1.27 1.27)
+				)
+			)
+		)
+		(property "Footprint" ""
+			(at 102.87 96.52 0)
+			(hide yes)
+			(show_name no)
+			(do_not_autoplace no)
+			(effects
+				(font
+					(size 1.27 1.27)
+				)
+			)
+		)
+		(property "Datasheet" ""
+			(at 102.87 96.52 0)
+			(hide yes)
+			(show_name no)
+			(do_not_autoplace no)
+			(effects
+				(font
+					(size 1.27 1.27)
+				)
+			)
+		)
+		(property "Description" "Special symbol for telling ERC where power comes from"
+			(at 102.87 96.52 0)
+			(hide yes)
+			(show_name no)
+			(do_not_autoplace no)
+			(effects
+				(font
+					(size 1.27 1.27)
+				)
+			)
+		)
+		(pin "1"
+		)
+		(instances
+			(project "tnu_pcb_pic40"
+				(path "/a3fd5e7d-0cea-44a9-a82d-5c7b53d9d25b/ad02958a-2d73-4242-8533-95aa22a85c5d"
+					(reference "#FLG02")
+					(unit 1)
+				)
+			)
+		)
+	)
+	(symbol
+		(lib_id "power:PWR_FLAG")
+		(at 60.96 50.8 0)
+		(unit 1)
+		(body_style 1)
+		(exclude_from_sim no)
+		(in_bom yes)
+		(on_board yes)
+		(in_pos_files yes)
+		(dnp no)
+		(fields_autoplaced yes)
+		(property "Reference" "#FLG03"
+			(at 60.96 48.895 0)
+			(hide yes)
+			(show_name no)
+			(do_not_autoplace no)
+			(effects
+				(font
+					(size 1.27 1.27)
+				)
+			)
+		)
+		(property "Value" "PWR_FLAG"
+			(at 60.96 46.99 0)
+			(show_name no)
+			(do_not_autoplace no)
+			(effects
+				(font
+					(size 1.27 1.27)
+				)
+			)
+		)
+		(property "Footprint" ""
+			(at 60.96 50.8 0)
+			(hide yes)
+			(show_name no)
+			(do_not_autoplace no)
+			(effects
+				(font
+					(size 1.27 1.27)
+				)
+			)
+		)
+		(property "Datasheet" ""
+			(at 60.96 50.8 0)
+			(hide yes)
+			(show_name no)
+			(do_not_autoplace no)
+			(effects
+				(font
+					(size 1.27 1.27)
+				)
+			)
+		)
+		(property "Description" "Special symbol for telling ERC where power comes from"
+			(at 60.96 50.8 0)
+			(hide yes)
+			(show_name no)
+			(do_not_autoplace no)
+			(effects
+				(font
+					(size 1.27 1.27)
+				)
+			)
+		)
+		(pin "1"
+		)
+		(instances
+			(project "tnu_pcb_pic40"
+				(path "/a3fd5e7d-0cea-44a9-a82d-5c7b53d9d25b/ad02958a-2d73-4242-8533-95aa22a85c5d"
+					(reference "#FLG03")
+					(unit 1)
+				)

Commit message: Connect USB UART via sheet pins; add MCLRn labels
Root: USB_TXD/USB_RXD/USB_RST hierarchical labels -> local labels (same
position and UUID); add sheet pins USB_TXD (input) and USB_RXD (output)
on the Microcontroller sheet symbol with wire stubs and local labels.
Microcontroller: USB_TXD shape input, USB_RXD shape output; MCLRn labels
join U3.1/R7/TP1 with J5.1/SW1.
/USB_TXD = U1.20 + U3.26, /USB_RXD = U1.4 + U3.25, MCLRn = U3.1, R7.2,
TP1, J5.1, SW1.1.
ERC 9 -> 1 (U4 footprint-filter warning only). DRC 84 + 152 unconnected;
parity 10 -> 20 (net renames, cleared by Update PCB from Schematic).

Co-Authored-By: Claude Opus 5.5 <noreply@anthropic.com>
Connections:
- net MCLRn: now reaches J5.1 (Pin_1), SW1.1
- net MCLRn: now also R7.2, TP1.1, U3.1 (~{MCLR}/VPP)
Changed lines of the file:
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@@
+		)
+	)
+	(label "MCLRn"
+		(at 110.49 58.42 0)
+		(effects
+			(font
+				(size 1.27 1.27)
+			)
+			(justify left bottom)
+		)
+	)
+	(label "MCLRn"
+		(at 90.17 90.17 0)
+		(effects
+			(font
+				(size 1.27 1.27)
+			)
+			(justify left bottom)
 		)
 	)
 	(hierarchical_label "USB_RXD"
-		(shape input)
+		(shape output)
 		(at 207.01 69.85 0)
 		(effects
@@
 	)
 	(hierarchical_label "USB_TXD"
-		(shape output)
+		(shape input)
 		(at 208.28 78.74 0)
 		(effects

Commit message: Fix supply test points: TP16/TP19 on VCC, TP18/TP21 on GND
Per the Cadence PDF: rename TP21 -> TP16 (VCC) and TP44 -> TP18 (GND);
add TP21 on GND (copy of TP18) wired to the U3 pin 12 ground corner.
ERC 1 (U4 warning, unchanged). DRC 84 + 152 unconnected; parity 20 -> 24
(TP renames, cleared by Update PCB from Schematic).

Co-Authored-By: Claude Opus 5.5 <noreply@anthropic.com>
Parts:
- added TP21: TP, TestPoint:TestPoint_Pad_D1.0mm, symbol Connector:TestPoint
- renumbered TP21 to TP16, TP44 to TP18
Connections:
- net GND: now also TP21.1
Changed lines of the file:
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@@
 	(paper "A4")
 	(junction
+		(at 148.59 119.38)
+		(diameter 0)
+		(color 0 0 0 0)
+	)
+	(junction
 		(at 151.13 119.38)
 		(diameter 0)
@@
 	(wire
 		(pts
+			(xy 148.59 119.38) (xy 143.51 119.38)
+		)
+		(stroke
+			(width 0)
+			(type default)
+		)
+	)
+	(wire
+		(pts
+			(xy 143.51 119.38) (xy 143.51 120.65)
+		)
+		(stroke
+			(width 0)
+			(type default)
+		)
+	)
+	(wire
+		(pts
 			(xy 49.53 34.29) (xy 102.87 34.29)
 		)
@@
 		(in_pos_files yes)
 		(dnp no)
-		(property "Reference" "TP21"
+		(property "Reference" "TP16"
 			(at 154.432 44.45 90)
 			(show_name no)
@@
 			(project "tnu_pcb_pic40"
 				(path "/a3fd5e7d-0cea-44a9-a82d-5c7b53d9d25b/ad02958a-2d73-4242-8533-95aa22a85c5d"
-					(reference "TP21")
+					(reference "TP16")
 					(unit 1)
 				)
@@
 		(in_pos_files yes)
 		(dnp no)
-		(property "Reference" "TP44"
+		(property "Reference" "TP18"
 			(at 147.574 124.206 0)
 			(show_name no)
@@
 			(project "tnu_pcb_pic40"
 				(path "/a3fd5e7d-0cea-44a9-a82d-5c7b53d9d25b/ad02958a-2d73-4242-8533-95aa22a85c5d"
-					(reference "TP44")
+					(reference "TP18")
+					(unit 1)
+				)
+			)
+		)
+	)
+	(symbol
+		(lib_id "Connector:TestPoint")
+		(at 143.51 120.65 180)
+		(unit 1)
+		(body_style 1)
+		(exclude_from_sim no)
+		(in_bom yes)
+		(on_board yes)
+		(in_pos_files yes)
+		(dnp no)
+		(property "Reference" "TP21"
+			(at 139.954 124.206 0)
+			(show_name no)
+			(do_not_autoplace no)
+			(effects
+				(font
+					(size 1.27 1.27)
+				)
+			)
+		)
+		(property "Value" "TP"
+			(at 140.97 123.952 90)
+			(hide yes)
+			(show_name no)
+			(do_not_autoplace no)
+			(effects
+				(font
+					(size 1.27 1.27)
+				)
+			)
+		)
+		(property "Footprint" "TestPoint:TestPoint_Pad_D1.0mm"
+			(at 138.43 120.65 0)
+			(hide yes)
+			(show_name no)
+			(do_not_autoplace no)
+			(effects
+				(font
+					(size 1.27 1.27)
+				)
+			)
+		)
+		(property "Datasheet" ""
+			(at 138.43 120.65 0)
+			(hide yes)
+			(show_name no)
+			(do_not_autoplace no)
+			(effects
+				(font
+					(size 1.27 1.27)
+				)
+			)
+		)
+		(property "Description" "TEST POINT PC COMPACT .063\"D BLK"
+			(at 143.51 120.65 0)
+			(hide yes)
+			(show_name no)
+			(do_not_autoplace no)
+			(effects
+				(font
+					(size 1.27 1.27)
+				)
+			)
+		)
+		(property "Manufacturer" "Keystone"
+			(at 143.51 120.65 0)
+			(hide yes)
+			(show_name no)
+			(do_not_autoplace no)
+			(effects
+				(font
+					(size 1.27 1.27)
+				)
+			)
+		)
+		(property "Manufacturer_PartNum" "5006"
+			(at 143.51 120.65 0)
+			(hide yes)
+			(show_name no)
+			(do_not_autoplace no)
+			(effects
+				(font
+					(size 1.27 1.27)
+				)
+			)
+		)
+		(property "Manufacturer2" ""
+			(at 143.51 120.65 0)
+			(hide yes)
+			(show_name no)
+			(do_not_autoplace no)
+			(effects
+				(font
+					(size 1.27 1.27)
+				)
+			)
+		)
+		(property "Manufacturer2_PartNum" ""
+			(at 143.51 120.65 0)
+			(hide yes)
+			(show_name no)
+			(do_not_autoplace no)
+			(effects
+				(font
+					(size 1.27 1.27)
+				)
+			)
+		)
+		(property "Distributor" "Digikey"
+			(at 143.51 120.65 0)
+			(hide yes)
+			(show_name no)
+			(do_not_autoplace no)
+			(effects
+				(font
+					(size 1.27 1.27)
+				)
+			)
+		)
+		(property "Distributor_PartNum" "5006K-ND"
+			(at 143.51 120.65 0)
+			(hide yes)
+			(show_name no)
+			(do_not_autoplace no)
+			(effects
+				(font
+					(size 1.27 1.27)
+				)
+			)
+		)
+		(property "Distributor2" ""
+			(at 143.51 120.65 0)
+			(hide yes)
+			(show_name no)
+			(do_not_autoplace no)
+			(effects
+				(font
+					(size 1.27 1.27)
+				)
+			)
+		)
+		(property "Distributor2_PartNum" ""
+			(at 143.51 120.65 0)
+			(hide yes)
+			(show_name no)
+			(do_not_autoplace no)
+			(effects
+				(font
+					(size 1.27 1.27)
+				)
+			)
+		)
+		(pin "1"
+		)
+		(instances
+			(project "tnu_pcb_pic40"
+				(path "/a3fd5e7d-0cea-44a9-a82d-5c7b53d9d25b/ad02958a-2d73-4242-8533-95aa22a85c5d"
+					(reference "TP21")
 					(unit 1)
 				)

Commit message: Add tnu footprint library; use pin header footprints for test points
tnu.pretty/TestPoint_PinHeader_1x01_P2.54mm: copy of KiCad
PinHeader_1x01_P2.54mm_Vertical (1.7 mm rect pad, 1.0 mm drill, origin on
pad) with a 2.54 x 2.54 mm courtyard, no silkscreen (Reference on F.Fab),
KiLib_Generator field removed. fp-lib-table: tnu -> ${KIPRJMOD}/tnu.pretty.
Footprint field of TP1-TP36 and P1-P19 (55 symbols) set to
tnu:TestPoint_PinHeader_1x01_P2.54mm; no other schematic change.
ERC 1 (U4). PCB not updated yet.

Co-Authored-By: Claude Opus 5.5 <noreply@anthropic.com>
Parts:
- P1, P11, P12, P13, P14, P15, P16, P17, P18, P19, P2, P3, P4, P5, P6, TP1, TP10, TP11, TP12, TP13, TP14, TP15, TP16, TP17, TP18, TP19, TP2, TP20, TP21, TP22, TP23, TP24, TP25, TP26, TP27, TP28, TP29, TP3, TP30, TP31, TP32, TP33, TP34, TP35, TP36, TP4, TP5, TP6, TP7, TP8, TP9: footprint TestPoint:TestPoint_Pad_D1.0mm -> tnu:TestPoint_PinHeader_1x01_P2.54mm
Changed lines of the file:
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@@
 			)
 		)
-		(property "Footprint" "TestPoint:TestPoint_Pad_D1.0mm"
+		(property "Footprint" "tnu:TestPoint_PinHeader_1x01_P2.54mm"
 			(at 39.37 116.84 0)
 			(hide yes)
@@
 			)
 		)
-		(property "Footprint" "TestPoint:TestPoint_Pad_D1.0mm"
+		(property "Footprint" "tnu:TestPoint_PinHeader_1x01_P2.54mm"
 			(at 157.48 46.99 0)
 			(hide yes)
@@
 			)
 		)
-		(property "Footprint" "TestPoint:TestPoint_Pad_D1.0mm"
+		(property "Footprint" "tnu:TestPoint_PinHeader_1x01_P2.54mm"
 			(at 185.42 109.22 0)
 			(hide yes)
@@
 			)
 		)
-		(property "Footprint" "TestPoint:TestPoint_Pad_D1.0mm"
+		(property "Footprint" "tnu:TestPoint_PinHeader_1x01_P2.54mm"
 			(at 121.92 91.44 0)
 			(hide yes)
@@
 			)
 		)
-		(property "Footprint" "TestPoint:TestPoint_Pad_D1.0mm"
+		(property "Footprint" "tnu:TestPoint_PinHeader_1x01_P2.54mm"
 			(at 146.05 120.65 0)
 			(hide yes)
@@
 			)
 		)
-		(property "Footprint" "TestPoint:TestPoint_Pad_D1.0mm"
+		(property "Footprint" "tnu:TestPoint_PinHeader_1x01_P2.54mm"
 			(at 39.37 111.76 0)
 			(hide yes)
@@
 			)
 		)
-		(property "Footprint" "TestPoint:TestPoint_Pad_D1.0mm"
+		(property "Footprint" "tnu:TestPoint_PinHeader_1x01_P2.54mm"
 			(at 39.37 77.47 0)
 			(hide yes)
@@
 			)
 		)
-		(property "Footprint" "TestPoint:TestPoint_Pad_D1.0mm"
+		(property "Footprint" "tnu:TestPoint_PinHeader_1x01_P2.54mm"
 			(at 39.37 87.63 0)
 			(hide yes)
@@
 			)
 		)
-		(property "Footprint" "TestPoint:TestPoint_Pad_D1.0mm"
+		(property "Footprint" "tnu:TestPoint_PinHeader_1x01_P2.54mm"
 			(at 185.42 68.58 0)
 			(hide yes)
@@
 			)
 		)
-		(property "Footprint" "TestPoint:TestPoint_Pad_D1.0mm"
+		(property "Footprint" "tnu:TestPoint_PinHeader_1x01_P2.54mm"
 			(at 121.92 83.82 0)
 			(hide yes)
@@
 			)
 		)
-		(property "Footprint" "TestPoint:TestPoint_Pad_D1.0mm"
+		(property "Footprint" "tnu:TestPoint_PinHeader_1x01_P2.54mm"
 			(at 39.37 96.52 0)
 			(hide yes)
@@
 			)
 		)
-		(property "Footprint" "TestPoint:TestPoint_Pad_D1.0mm"
+		(property "Footprint" "tnu:TestPoint_PinHeader_1x01_P2.54mm"
 			(at 152.4 46.99 0)
 			(hide yes)
@@
 			)
 		)
-		(property "Footprint" "TestPoint:TestPoint_Pad_D1.0mm"
+		(property "Footprint" "tnu:TestPoint_PinHeader_1x01_P2.54mm"
 			(at 121.92 63.5 0)
 			(hide yes)
@@
 			)
 		)
-		(property "Footprint" "TestPoint:TestPoint_Pad_D1.0mm"
+		(property "Footprint" "tnu:TestPoint_PinHeader_1x01_P2.54mm"
 			(at 172.72 30.48 0)
 			(hide yes)
@@
 			)
 		)
-		(property "Footprint" "TestPoint:TestPoint_Pad_D1.0mm"
+		(property "Footprint" "tnu:TestPoint_PinHeader_1x01_P2.54mm"
 			(at 121.92 86.36 0)
 			(hide yes)
@@
 			)
 		)
-		(property "Footprint" "TestPoint:TestPoint_Pad_D1.0mm"
+		(property "Footprint" "tnu:TestPoint_PinHeader_1x01_P2.54mm"
 			(at 121.92 96.52 0)
 			(hide yes)
@@
 			)
 		)
-		(property "Footprint" "TestPoint:TestPoint_Pad_D1.0mm"
+		(property "Footprint" "tnu:TestPoint_PinHeader_1x01_P2.54mm"
 			(at 121.92 60.96 0)
 			(hide yes)
@@
 			)
 		)
-		(property "Footprint" "TestPoint:TestPoint_Pad_D1.0mm"
+		(property "Footprint" "tnu:TestPoint_PinHeader_1x01_P2.54mm"
 			(at 121.92 93.98 0)
 			(hide yes)
@@
 			)
 		)
-		(property "Footprint" "TestPoint:TestPoint_Pad_D1.0mm"
+		(property "Footprint" "tnu:TestPoint_PinHeader_1x01_P2.54mm"
 			(at 185.42 114.3 0)
 			(hide yes)
@@
 			)
 		)
-		(property "Footprint" "TestPoint:TestPoint_Pad_D1.0mm"
+		(property "Footprint" "tnu:TestPoint_PinHeader_1x01_P2.54mm"
 			(at 185.42 111.76 0)
 			(hide yes)
@@
 			)
 		)
-		(property "Footprint" "TestPoint:TestPoint_Pad_D1.0mm"
+		(property "Footprint" "tnu:TestPoint_PinHeader_1x01_P2.54mm"
 			(at 185.42 104.14 0)
 			(hide yes)
@@
 			)
 		)
-		(property "Footprint" "TestPoint:TestPoint_Pad_D1.0mm"
+		(property "Footprint" "tnu:TestPoint_PinHeader_1x01_P2.54mm"
 			(at 185.42 96.52 0)
 			(hide yes)
@@
 			)
 		)
-		(property "Footprint" "TestPoint:TestPoint_Pad_D1.0mm"
+		(property "Footprint" "tnu:TestPoint_PinHeader_1x01_P2.54mm"
 			(at 39.37 106.68 0)
 			(hide yes)
@@
 			)
 		)
-		(property "Footprint" "TestPoint:TestPoint_Pad_D1.0mm"
+		(property "Footprint" "tnu:TestPoint_PinHeader_1x01_P2.54mm"
 			(at 185.42 86.36 0)
 			(hide yes)
@@
 			)
 		)
-		(property "Footprint" "TestPoint:TestPoint_Pad_D1.0mm"
+		(property "Footprint" "tnu:TestPoint_PinHeader_1x01_P2.54mm"
 			(at 39.37 91.44 0)
 			(hide yes)
@@
 			)
 		)
-		(property "Footprint" "TestPoint:TestPoint_Pad_D1.0mm"
+		(property "Footprint" "tnu:TestPoint_PinHeader_1x01_P2.54mm"
 			(at 203.2 81.28 0)
 			(hide yes)
@@
 			)
 		)
-		(property "Footprint" "TestPoint:TestPoint_Pad_D1.0mm"
+		(property "Footprint" "tnu:TestPoint_PinHeader_1x01_P2.54mm"
 			(at 101.6 54.61 0)
 			(hide yes)
@@
 			)
 		)
-		(property "Footprint" "TestPoint:TestPoint_Pad_D1.0mm"
+		(property "Footprint" "tnu:TestPoint_PinHeader_1x01_P2.54mm"
 			(at 121.92 66.04 0)
 			(hide yes)
@@
 			)
 		)
-		(property "Footprint" "TestPoint:TestPoint_Pad_D1.0mm"
+		(property "Footprint" "tnu:TestPoint_PinHeader_1x01_P2.54mm"
 			(at 121.92 88.9 0)
 			(hide yes)
@@
 			)
 		)
-		(property "Footprint" "TestPoint:TestPoint_Pad_D1.0mm"
+		(property "Footprint" "tnu:TestPoint_PinHeader_1x01_P2.54mm"
 			(at 39.37 121.92 0)
 			(hide yes)
@@
 			)
 		)
-		(property "Footprint" "TestPoint:TestPoint_Pad_D1.0mm"
+		(property "Footprint" "tnu:TestPoint_PinHeader_1x01_P2.54mm"
 			(at 185.42 66.04 0)
 			(hide yes)
@@
 			)
 		)
-		(property "Footprint" "TestPoint:TestPoint_Pad_D1.0mm"
+		(property "Footprint" "tnu:TestPoint_PinHeader_1x01_P2.54mm"
 			(at 185.42 63.5 0)
 			(hide yes)
@@
 			)
 		)
-		(property "Footprint" "TestPoint:TestPoint_Pad_D1.0mm"
+		(property "Footprint" "tnu:TestPoint_PinHeader_1x01_P2.54mm"
 			(at 39.37 132.08 0)
 			(hide yes)
@@
 			)
 		)
-		(property "Footprint" "TestPoint:TestPoint_Pad_D1.0mm"
+		(property "Footprint" "tnu:TestPoint_PinHeader_1x01_P2.54mm"
 			(at 185.42 73.66 0)
 			(hide yes)
@@
 			)
 		)
-		(property "Footprint" "TestPoint:TestPoint_Pad_D1.0mm"
+		(property "Footprint" "tnu:TestPoint_PinHeader_1x01_P2.54mm"
 			(at 121.92 71.12 0)
 			(hide yes)
@@
 			)
 		)
-		(property "Footprint" "TestPoint:TestPoint_Pad_D1.0mm"
+		(property "Footprint" "tnu:TestPoint_PinHeader_1x01_P2.54mm"
 			(at 185.42 88.9 0)
 			(hide yes)
@@
 			)
 		)
-		(property "Footprint" "TestPoint:TestPoint_Pad_D1.0mm"
+		(property "Footprint" "tnu:TestPoint_PinHeader_1x01_P2.54mm"
 			(at 40.64 45.72 0)
 			(hide yes)
@@
 			)
 		)
-		(property "Footprint" "TestPoint:TestPoint_Pad_D1.0mm"
+		(property "Footprint" "tnu:TestPoint_PinHeader_1x01_P2.54mm"
 			(at 185.42 101.6 0)
 			(hide yes)
@@
 			)
 		)
-		(property "Footprint" "TestPoint:TestPoint_Pad_D1.0mm"
+		(property "Footprint" "tnu:TestPoint_PinHeader_1x01_P2.54mm"
 			(at 121.92 68.58 0)
 			(hide yes)
@@
 			)
 		)
-		(property "Footprint" "TestPoint:TestPoint_Pad_D1.0mm"
+		(property "Footprint" "tnu:TestPoint_PinHeader_1x01_P2.54mm"
 			(at 138.43 120.65 0)
 			(hide yes)
@@
 			)
 		)
-		(property "Footprint" "TestPoint:TestPoint_Pad_D1.0mm"
+		(property "Footprint" "tnu:TestPoint_PinHeader_1x01_P2.54mm"
 			(at 185.42 71.12 0)
 			(hide yes)
@@
 			)
 		)
-		(property "Footprint" "TestPoint:TestPoint_Pad_D1.0mm"
+		(property "Footprint" "tnu:TestPoint_PinHeader_1x01_P2.54mm"
 			(at 39.37 127 0)
 			(hide yes)
@@
 			)
 		)
-		(property "Footprint" "TestPoint:TestPoint_Pad_D1.0mm"
+		(property "Footprint" "tnu:TestPoint_PinHeader_1x01_P2.54mm"
 			(at 185.42 91.44 0)
 			(hide yes)
@@
 			)
 		)
-		(property "Footprint" "TestPoint:TestPoint_Pad_D1.0mm"
+		(property "Footprint" "tnu:TestPoint_PinHeader_1x01_P2.54mm"
 			(at 181.61 20.32 0)
 			(hide yes)
@@
 			)
 		)
-		(property "Footprint" "TestPoint:TestPoint_Pad_D1.0mm"
+		(property "Footprint" "tnu:TestPoint_PinHeader_1x01_P2.54mm"
 			(at 185.42 93.98 0)
 			(hide yes)
@@
 			)
 		)
-		(property "Footprint" "TestPoint:TestPoint_Pad_D1.0mm"
+		(property "Footprint" "tnu:TestPoint_PinHeader_1x01_P2.54mm"
 			(at 121.92 58.42 0)
 			(hide yes)
@@
 			)
 		)
-		(property "Footprint" "TestPoint:TestPoint_Pad_D1.0mm"
+		(property "Footprint" "tnu:TestPoint_PinHeader_1x01_P2.54mm"
 			(at 39.37 82.55 0)
 			(hide yes)
@@
 			)
 		)
-		(property "Footprint" "TestPoint:TestPoint_Pad_D1.0mm"
+		(property "Footprint" "tnu:TestPoint_PinHeader_1x01_P2.54mm"
 			(at 203.2 78.74 0)
 			(hide yes)
@@
 			)
 		)
-		(property "Footprint" "TestPoint:TestPoint_Pad_D1.0mm"
+		(property "Footprint" "tnu:TestPoint_PinHeader_1x01_P2.54mm"
 			(at 185.42 99.06 0)
 			(hide yes)
@@
 			)
 		)
-		(property "Footprint" "TestPoint:TestPoint_Pad_D1.0mm"
+		(property "Footprint" "tnu:TestPoint_PinHeader_1x01_P2.54mm"
 			(at 39.37 101.6 0)
 			(hide yes)
@@
 			)
 		)
-		(property "Footprint" "TestPoint:TestPoint_Pad_D1.0mm"
+		(property "Footprint" "tnu:TestPoint_PinHeader_1x01_P2.54mm"
 			(at 185.42 76.2 0)
 			(hide yes)
