File: tnu_pcb_pic40.kicad_sch (KiCad schematic)
At the start: 23 parts, among them CN1 USB_B_receptacle, P10 TP, P7 TP, P8 TP, P9 TP, U1 FT231XS-R

Commit message: ERC cleanup: NC flags, PWR_FLAGs, remove stray #PWR012, usb->GND
- No-connect flags on FT231XS U1 pins 1 (DTR), 5 (RI), 7 (DSR), 8 (DCD).
- Delete floating "usb" ground symbol #PWR012.
- Change the 7 remaining "usb" (power:GNDD) grounds to power:GND; same net.
- PWR_FLAG on VCC5_USB (#FLG01), VCC (#FLG02) and the J1 input rail
  (#FLG03); two wires split at the flag points, with junctions.
- Re-enable the "footprint doesn't match footprint filters" ERC check.

ERC 20 -> 9 (8 remaining are the Step 2 USB UART issues, plus 1 new
footprint_filter warning on U4, already in the footprint fix list).
DRC unchanged: 84 + 152 unconnected + 8 known parity issues.

Co-Authored-By: Claude Opus 5.5 <noreply@anthropic.com>
Connections:
- no-connect marks 0 -> 4
Changed lines of the file:
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@@
 	(paper "A4")
 	(junction
+		(at 92.71 40.64)
+		(diameter 0)
+		(color 0 0 0 0)
+	)
+	(junction
 		(at 69.85 73.66)
 		(diameter 0)
@@
 		(color 0 0 0 0)
 	)
+	(no_connect
+		(at 166.37 74.93)
+	)
+	(no_connect
+		(at 166.37 82.55)
+	)
+	(no_connect
+		(at 166.37 77.47)
+	)
+	(no_connect
+		(at 166.37 80.01)
+	)
 	(wire
 		(pts
@@
 	(wire
 		(pts
-			(xy 85.09 40.64) (xy 100.33 40.64)
+			(xy 85.09 40.64) (xy 92.71 40.64)
+		)
+		(stroke
+			(width 0)
+			(type default)
+		)
+	)
+	(wire
+		(pts
+			(xy 92.71 40.64) (xy 100.33 40.64)
 		)
 		(stroke
@@
 	)
 	(symbol
-		(lib_id "power:GNDD")
+		(lib_id "power:GND")
 		(at 33.02 96.52 0)
 		(unit 1)
@@
 			)
 		)
-		(property "Value" "usb"
+		(property "Value" "GND"
 			(at 33.02 100.33 0)
 			(show_name no)
@@
 			)
 		)
-		(property "Description" "Power symbol creates a global label with name \"GNDD\" , digital ground"
+		(property "Description" "Power symbol creates a global label with name \"GND\" , ground"
 			(at 33.02 96.52 0)
 			(hide yes)
@@
 	)
 	(symbol
-		(lib_id "power:GNDD")
+		(lib_id "power:GND")
 		(at 69.85 90.17 0)
 		(unit 1)
@@
 			)
 		)
-		(property "Value" "usb"
+		(property "Value" "GND"
 			(at 69.85 93.98 0)
 			(show_name no)
@@
 			)
 		)
-		(property "Description" "Power symbol creates a global label with name \"GNDD\" , digital ground"
+		(property "Description" "Power symbol creates a global label with name \"GND\" , ground"
 			(at 69.85 90.17 0)
 			(hide yes)
@@
 	)
 	(symbol
-		(lib_id "power:GNDD")
+		(lib_id "power:GND")
 		(at 157.48 107.95 0)
 		(unit 1)
@@
 			)
 		)
-		(property "Value" "usb"
+		(property "Value" "GND"
 			(at 157.48 111.76 0)
 			(show_name no)
@@
 			)
 		)
-		(property "Description" "Power symbol creates a global label with name \"GNDD\" , digital ground"
+		(property "Description" "Power symbol creates a global label with name \"GND\" , ground"
 			(at 157.48 107.95 0)
 			(hide yes)
@@
 	)
 	(symbol
-		(lib_id "power:GNDD")
+		(lib_id "power:GND")
 		(at 82.55 90.17 0)
 		(unit 1)
@@
 			)
 		)
-		(property "Value" "usb"
+		(property "Value" "GND"
 			(at 82.55 93.98 0)
 			(show_name no)
@@
 			)
 		)
-		(property "Description" "Power symbol creates a global label with name \"GNDD\" , digital ground"
+		(property "Description" "Power symbol creates a global label with name \"GND\" , ground"
 			(at 82.55 90.17 0)
 			(hide yes)
@@
 	)
 	(symbol
-		(lib_id "power:GNDD")
+		(lib_id "power:GND")
 		(at 48.26 55.88 0)
 		(unit 1)
@@
 			)
 		)
-		(property "Value" "usb"
+		(property "Value" "GND"
 			(at 48.26 59.69 0)
 			(show_name no)
@@
 			)
 		)
-		(property "Description" "Power symbol creates a global label with name \"GNDD\" , digital ground"
+		(property "Description" "Power symbol creates a global label with name \"GND\" , ground"
 			(at 48.26 55.88 0)
 			(hide yes)
@@
 	)
 	(symbol
-		(lib_id "power:GNDD")
-		(at 41.91 154.94 0)
-		(unit 1)
-		(body_style 1)
-		(exclude_from_sim no)
-		(in_bom yes)
-		(on_board yes)
-		(in_pos_files yes)
-		(dnp no)
-		(fields_autoplaced yes)
-		(property "Reference" "#PWR012"
-			(at 41.91 161.29 0)
-			(hide yes)
-			(show_name no)
-			(do_not_autoplace no)
-			(effects
-				(font
-					(size 1.27 1.27)
-				)
-			)
-		)
-		(property "Value" "usb"
-			(at 41.91 158.75 0)
-			(show_name no)
-			(do_not_autoplace no)
-			(effects
-				(font
-					(size 1.27 1.27)
-				)
-			)
-		)
-		(property "Footprint" ""
-			(at 41.91 154.94 0)
-			(hide yes)
-			(show_name no)
-			(do_not_autoplace no)
-			(effects
-				(font
-					(size 1.27 1.27)
-				)
-			)
-		)
-		(property "Datasheet" ""
-			(at 41.91 154.94 0)
-			(hide yes)
-			(show_name no)
-			(do_not_autoplace no)
-			(effects
-				(font
-					(size 1.27 1.27)
-				)
-			)
-		)
-		(property "Description" "Power symbol creates a global label with name \"GNDD\" , digital ground"
-			(at 41.91 154.94 0)
-			(hide yes)
-			(show_name no)
-			(do_not_autoplace no)
-			(effects
-				(font
-					(size 1.27 1.27)
-				)
-			)
-		)
-		(property "Manufacturer" ""
-			(at 41.91 154.94 0)
-			(hide yes)
-			(show_name no)
-			(do_not_autoplace no)
-			(effects
-				(font
-					(size 1.27 1.27)
-				)
-			)
-		)
-		(property "Manufacturer_PartNum" ""
-			(at 41.91 154.94 0)
-			(hide yes)
-			(show_name no)
-			(do_not_autoplace no)
-			(effects
-				(font
-					(size 1.27 1.27)
-				)
-			)
-		)
-		(property "Manufacturer2" ""
-			(at 41.91 154.94 0)
-			(hide yes)
-			(show_name no)
-			(do_not_autoplace no)
-			(effects
-				(font
-					(size 1.27 1.27)
-				)
-			)
-		)
-		(property "Manufacturer2_PartNum" ""
-			(at 41.91 154.94 0)
-			(hide yes)
-			(show_name no)
-			(do_not_autoplace no)
-			(effects
-				(font
-					(size 1.27 1.27)
-				)
-			)
-		)
-		(property "Distributor" ""
-			(at 41.91 154.94 0)
-			(hide yes)
-			(show_name no)
-			(do_not_autoplace no)
-			(effects
-				(font
-					(size 1.27 1.27)
-				)
-			)
-		)
-		(property "Distributor_PartNum" ""
-			(at 41.91 154.94 0)
-			(hide yes)
-			(show_name no)
-			(do_not_autoplace no)
-			(effects
-				(font
-					(size 1.27 1.27)
-				)
-			)
-		)
-		(property "Distributor2" ""
-			(at 41.91 154.94 0)
-			(hide yes)
-			(show_name no)
-			(do_not_autoplace no)
-			(effects
-				(font
-					(size 1.27 1.27)
-				)
-			)
-		)
-		(property "Distributor2_PartNum" ""
-			(at 41.91 154.94 0)
-			(hide yes)
-			(show_name no)
-			(do_not_autoplace no)
-			(effects
-				(font
-					(size 1.27 1.27)
-				)
-			)
-		)
-		(pin "1"
-		)
-		(instances
-			(project "tnu_pcb_pic40"
-				(path "/a3fd5e7d-0cea-44a9-a82d-5c7b53d9d25b"
-					(reference "#PWR012")
-					(unit 1)
-				)
-			)
-		)
-	)
-	(symbol
-		(lib_id "power:GNDD")
+		(lib_id "power:GND")
 		(at 100.33 49.53 0)
 		(unit 1)
@@
 			)
 		)
-		(property "Value" "usb"
+		(property "Value" "GND"
 			(at 100.33 53.34 0)
 			(show_name no)
@@
 			)
 		)
-		(property "Description" "Power symbol creates a global label with name \"GNDD\" , digital ground"
+		(property "Description" "Power symbol creates a global label with name \"GND\" , ground"
 			(at 100.33 49.53 0)
 			(hide yes)
@@
 	)
 	(symbol
-		(lib_id "power:GNDD")
+		(lib_id "power:GND")
 		(at 101.6 142.24 0)
 		(unit 1)
@@
 			)
 		)
-		(property "Value" "usb"
+		(property "Value" "GND"
 			(at 101.6 146.05 0)
 			(show_name no)
@@
 			)
 		)
-		(property "Description" "Power symbol creates a global label with name \"GNDD\" , digital ground"
+		(property "Description" "Power symbol creates a global label with name \"GND\" , ground"
 			(at 101.6 142.24 0)
 			(hide yes)
@@
 					(unit 1)
 				)
+			)
+		)
+	)
+	(symbol
+		(lib_id "power:PWR_FLAG")
+		(at 92.71 40.64 0)
+		(unit 1)
+		(body_style 1)
+		(exclude_from_sim no)
+		(in_bom yes)
+		(on_board yes)
+		(in_pos_files yes)
+		(dnp no)
+		(fields_autoplaced yes)
+		(property "Reference" "#FLG01"
+			(at 92.71 38.735 0)
+			(hide yes)
+			(show_name no)
+			(do_not_autoplace no)
+			(effects
+				(font
+					(size 1.27 1.27)
+				)
+			)
+		)
+		(property "Value" "PWR_FLAG"
+			(at 92.71 36.83 0)
+			(show_name no)
+			(do_not_autoplace no)
+			(effects
+				(font
+					(size 1.27 1.27)
+				)
+			)
+		)
+		(property "Footprint" ""
+			(at 92.71 40.64 0)
+			(hide yes)
+			(show_name no)
+			(do_not_autoplace no)
+			(effects
+				(font
+					(size 1.27 1.27)
+				)
+			)
+		)
+		(property "Datasheet" ""
+			(at 92.71 40.64 0)
+			(hide yes)
+			(show_name no)
+			(do_not_autoplace no)
+			(effects
+				(font
+					(size 1.27 1.27)
+				)
+			)
+		)
+		(property "Description" "Special symbol for telling ERC where power comes from"
+			(at 92.71 40.64 0)
+			(hide yes)
+			(show_name no)
+			(do_not_autoplace no)
+			(effects
+				(font
+					(size 1.27 1.27)
+				)
+			)
+		)
+		(pin "1"
+		)
+		(instances
+			(project "tnu_pcb_pic40"
+				(path "/a3fd5e7d-0cea-44a9-a82d-5c7b53d9d25b"
+					(reference "#FLG01")
+					(unit 1)
+				)

Commit message: Ground C5/C6 decoupling caps (#PWR012 was never connected in the import)
Add GND symbol, wires and junction under C5/C6 on the root sheet.
Net-(C5-Pad2) is gone; C5.2 and C6.2 are on GND. The microcontroller
sheet diff is KiCad re-sorting earlier hand-inserted items (order only).
ERC 9 (unchanged). DRC 84 + 152 unconnected; parity 8 -> 10 (C5/C6 pad 2,
cleared by Update PCB from Schematic).

Co-Authored-By: Claude Opus 5.5 <noreply@anthropic.com>
Connections:
- net GND: now also C5.2, C6.2
Changed lines of the file:
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@@
 	(paper "A4")
 	(junction
-		(at 92.71 40.64)
+		(at 43.18 148.59)
 		(diameter 0)
 		(color 0 0 0 0)
@@
 	)
 	(junction
+		(at 92.71 40.64)
+		(diameter 0)
+		(color 0 0 0 0)
+	)
+	(junction
 		(at 90.17 130.81)
 		(diameter 0)
@@
 	)
 	(no_connect
-		(at 166.37 74.93)
+		(at 166.37 80.01)
 	)
 	(no_connect
-		(at 166.37 82.55)
+		(at 166.37 74.93)
 	)
 	(no_connect
@@
 	)
 	(no_connect
-		(at 166.37 80.01)
+		(at 166.37 82.55)
 	)
 	(wire
@@
 	(wire
 		(pts
+			(xy 43.18 148.59) (xy 43.18 154.94)
+		)
+		(stroke
+			(width 0)
+			(type default)
+		)
+	)
+	(wire
+		(pts
 			(xy 151.13 38.1) (xy 151.13 57.15)
 		)
@@
 	(wire
 		(pts
-			(xy 92.71 40.64) (xy 100.33 40.64)
+			(xy 100.33 40.64) (xy 104.14 40.64)
 		)
 		(stroke
@@
 	(wire
 		(pts
-			(xy 100.33 40.64) (xy 104.14 40.64)
+			(xy 104.14 40.64) (xy 146.05 40.64)
 		)
 		(stroke
@@
 	(wire
 		(pts
-			(xy 104.14 40.64) (xy 146.05 40.64)
+			(xy 64.77 138.43) (xy 77.47 138.43)
 		)
 		(stroke
@@
 	(wire
 		(pts
-			(xy 64.77 138.43) (xy 77.47 138.43)
+			(xy 101.6 138.43) (xy 101.6 142.24)
 		)
 		(stroke
@@
 	(wire
 		(pts
-			(xy 101.6 138.43) (xy 101.6 142.24)
+			(xy 82.55 76.2) (xy 101.6 76.2)
 		)
 		(stroke
@@
 	(wire
 		(pts
-			(xy 82.55 76.2) (xy 101.6 76.2)
+			(xy 166.37 90.17) (xy 181.61 90.17)
 		)
 		(stroke
@@
 	(wire
 		(pts
-			(xy 166.37 90.17) (xy 181.61 90.17)
+			(xy 40.64 76.2) (xy 82.55 76.2)
 		)
 		(stroke
@@
 	(wire
 		(pts
-			(xy 40.64 76.2) (xy 82.55 76.2)
+			(xy 92.71 40.64) (xy 100.33 40.64)
 		)
 		(stroke
@@
 	(wire
 		(pts
+			(xy 43.18 148.59) (xy 41.91 148.59)
+		)
+		(stroke
+			(width 0)
+			(type default)
+		)
+	)
+	(wire
+		(pts
 			(xy 146.05 102.87) (xy 151.13 102.87)
 		)
@@
 	(wire
 		(pts
-			(xy 52.07 148.59) (xy 41.91 148.59)
+			(xy 52.07 148.59) (xy 43.18 148.59)
 		)
 		(stroke
@@
 	)
 	(symbol
+		(lib_id "power:PWR_FLAG")
+		(at 92.71 40.64 0)
+		(unit 1)
+		(body_style 1)
+		(exclude_from_sim no)
+		(in_bom yes)
+		(on_board yes)
+		(in_pos_files yes)
+		(dnp no)
+		(fields_autoplaced yes)
+		(property "Reference" "#FLG01"
+			(at 92.71 38.735 0)
+			(hide yes)
+			(show_name no)
+			(do_not_autoplace no)
+			(effects
+				(font
+					(size 1.27 1.27)
+				)
+			)
+		)
+		(property "Value" "PWR_FLAG"
+			(at 92.71 36.83 0)
+			(show_name no)
+			(do_not_autoplace no)
+			(effects
+				(font
+					(size 1.27 1.27)
+				)
+			)
+		)
+		(property "Footprint" ""
+			(at 92.71 40.64 0)
+			(hide yes)
+			(show_name no)
+			(do_not_autoplace no)
+			(effects
+				(font
+					(size 1.27 1.27)
+				)
+			)
+		)
+		(property "Datasheet" ""
+			(at 92.71 40.64 0)
+			(hide yes)
+			(show_name no)
+			(do_not_autoplace no)
+			(effects
+				(font
+					(size 1.27 1.27)
+				)
+			)
+		)
+		(property "Description" "Special symbol for telling ERC where power comes from"
+			(at 92.71 40.64 0)
+			(hide yes)
+			(show_name no)
+			(do_not_autoplace no)
+			(effects
+				(font
+					(size 1.27 1.27)
+				)
+			)
+		)
+		(pin "1"
+		)
+		(instances
+			(project "tnu_pcb_pic40"
+				(path "/a3fd5e7d-0cea-44a9-a82d-5c7b53d9d25b"
+					(reference "#FLG01")
+					(unit 1)
+				)
+			)
+		)
+	)
+	(symbol
 		(lib_id "Connector:USB_B")
 		(at 33.02 73.66 0)
@@
 	(symbol
 		(lib_id "power:GND")
+		(at 43.18 154.94 0)
+		(unit 1)
+		(body_style 1)
+		(exclude_from_sim no)
+		(in_bom yes)
+		(on_board yes)
+		(in_pos_files yes)
+		(dnp no)
+		(fields_autoplaced yes)
+		(property "Reference" "#PWR012"
+			(at 43.18 161.29 0)
+			(hide yes)
+			(show_name no)
+			(do_not_autoplace no)
+			(effects
+				(font
+					(size 1.27 1.27)
+				)
+			)
+		)
+		(property "Value" "GND"
+			(at 43.18 160.02 0)
+			(show_name no)
+			(do_not_autoplace no)
+			(effects
+				(font
+					(size 1.27 1.27)
+				)
+			)
+		)
+		(property "Footprint" ""
+			(at 43.18 154.94 0)
+			(hide yes)
+			(show_name no)
+			(do_not_autoplace no)
+			(effects
+				(font
+					(size 1.27 1.27)
+				)
+			)
+		)
+		(property "Datasheet" ""
+			(at 43.18 154.94 0)
+			(hide yes)
+			(show_name no)
+			(do_not_autoplace no)
+			(effects
+				(font
+					(size 1.27 1.27)
+				)
+			)
+		)
+		(property "Description" "Power symbol creates a global label with name \"GND\" , ground"
+			(at 43.18 154.94 0)
+			(hide yes)
+			(show_name no)
+			(do_not_autoplace no)
+			(effects
+				(font
+					(size 1.27 1.27)
+				)
+			)
+		)
+		(pin "1"
+		)
+		(instances
+			(project "tnu_pcb_pic40"
+				(path "/a3fd5e7d-0cea-44a9-a82d-5c7b53d9d25b"
+					(reference "#PWR012")
+					(unit 1)
+				)
+			)
+		)
+	)
+	(symbol
+		(lib_id "power:GND")
 		(at 157.48 107.95 0)
 		(unit 1)
@@
 					(unit 1)
 				)
-			)
-		)
-	)
-	(symbol
-		(lib_id "power:PWR_FLAG")
-		(at 92.71 40.64 0)
-		(unit 1)
-		(body_style 1)
-		(exclude_from_sim no)
-		(in_bom yes)
-		(on_board yes)
-		(in_pos_files yes)
-		(dnp no)
-		(fields_autoplaced yes)
-		(property "Reference" "#FLG01"
-			(at 92.71 38.735 0)
-			(hide yes)
-			(show_name no)
-			(do_not_autoplace no)
-			(effects
-				(font
-					(size 1.27 1.27)
-				)
-			)
-		)
-		(property "Value" "PWR_FLAG"
-			(at 92.71 36.83 0)
-			(show_name no)
-			(do_not_autoplace no)
-			(effects
-				(font
-					(size 1.27 1.27)
-				)
-			)
-		)
-		(property "Footprint" ""
-			(at 92.71 40.64 0)
-			(hide yes)
-			(show_name no)
-			(do_not_autoplace no)
-			(effects
-				(font
-					(size 1.27 1.27)
-				)
-			)
-		)
-		(property "Datasheet" ""
-			(at 92.71 40.64 0)
-			(hide yes)
-			(show_name no)
-			(do_not_autoplace no)
-			(effects
-				(font
-					(size 1.27 1.27)
-				)
-			)
-		)
-		(property "Description" "Special symbol for telling ERC where power comes from"
-			(at 92.71 40.64 0)
-			(hide yes)
-			(show_name no)
-			(do_not_autoplace no)
-			(effects
-				(font
-					(size 1.27 1.27)
-				)
-			)
-		)
-		(pin "1"
-		)
-		(instances
-			(project "tnu_pcb_pic40"
-				(path "/a3fd5e7d-0cea-44a9-a82d-5c7b53d9d25b"
-					(reference "#FLG01")
-					(unit 1)
-				)

Commit message: Connect USB UART via sheet pins; add MCLRn labels
Root: USB_TXD/USB_RXD/USB_RST hierarchical labels -> local labels (same
position and UUID); add sheet pins USB_TXD (input) and USB_RXD (output)
on the Microcontroller sheet symbol with wire stubs and local labels.
Microcontroller: USB_TXD shape input, USB_RXD shape output; MCLRn labels
join U3.1/R7/TP1 with J5.1/SW1.
/USB_TXD = U1.20 + U3.26, /USB_RXD = U1.4 + U3.25, MCLRn = U3.1, R7.2,
TP1, J5.1, SW1.1.
ERC 9 -> 1 (U4 footprint-filter warning only). DRC 84 + 152 unconnected;
parity 10 -> 20 (net renames, cleared by Update PCB from Schematic).

Co-Authored-By: Claude Opus 5.5 <noreply@anthropic.com>
Other:
- sheet Microcontroller ports: added USB_RXD, USB_TXD; removed none
Changed lines of the file:
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@@
 	(wire
 		(pts
+			(xy 165.1 231.14) (xy 165.1 226.06)
+		)
+		(stroke
+			(width 0)
+			(type default)
+		)
+	)
+	(wire
+		(pts
+			(xy 170.18 231.14) (xy 170.18 226.06)
+		)
+		(stroke
+			(width 0)
+			(type default)
+		)
+	)
+	(wire
+		(pts
 			(xy 201.93 139.7) (xy 201.93 140.97)
 		)
@@
 		)
 	)
-	(hierarchical_label "USB_TXD"
-		(shape output)
+	(label "USB_TXD"
 		(at 171.45 64.77 0)
 		(effects
@@
 				(size 1.27 1.27)
 			)
-			(justify left)
+			(justify left bottom)
 		)
 	)
-	(hierarchical_label "USB_RXD"
-		(shape input)
+	(label "USB_RXD"
 		(at 171.45 67.31 0)
 		(effects
@@
 				(size 1.27 1.27)
 			)
-			(justify left)
+			(justify left bottom)
 		)
 	)
-	(hierarchical_label "USB_RST"
-		(shape output)
+	(label "USB_RST"
 		(at 77.47 118.11 180)
 		(effects
@@
 				(size 1.27 1.27)
 			)
-			(justify right)
+			(justify right bottom)
+		)
+	)
+	(label "USB_TXD"
+		(at 165.1 226.06 90)
+		(effects
+			(font
+				(size 1.27 1.27)
+			)
+			(justify left bottom)
+		)
+	)
+	(label "USB_RXD"
+		(at 170.18 226.06 90)
+		(effects
+			(font
+				(size 1.27 1.27)
+			)
+			(justify left bottom)
 		)
 	)
@@
 			)
 		)
+		(pin "USB_TXD" input
+			(at 165.1 231.14 90)
+			(effects
+				(font
+					(size 1.27 1.27)
+				)
+				(justify right)
+			)
+		)
+		(pin "USB_RXD" output
+			(at 170.18 231.14 90)
+			(effects
+				(font
+					(size 1.27 1.27)
+				)
+				(justify right)
+			)
+		)

Commit message: Add tnu footprint library; use pin header footprints for test points
tnu.pretty/TestPoint_PinHeader_1x01_P2.54mm: copy of KiCad
PinHeader_1x01_P2.54mm_Vertical (1.7 mm rect pad, 1.0 mm drill, origin on
pad) with a 2.54 x 2.54 mm courtyard, no silkscreen (Reference on F.Fab),
KiLib_Generator field removed. fp-lib-table: tnu -> ${KIPRJMOD}/tnu.pretty.
Footprint field of TP1-TP36 and P1-P19 (55 symbols) set to
tnu:TestPoint_PinHeader_1x01_P2.54mm; no other schematic change.
ERC 1 (U4). PCB not updated yet.

Co-Authored-By: Claude Opus 5.5 <noreply@anthropic.com>
Parts:
- P10, P7, P8, P9: footprint TestPoint:TestPoint_Pad_D1.0mm -> tnu:TestPoint_PinHeader_1x01_P2.54mm
Changed lines of the file:
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@@
 			)
 		)
-		(property "Footprint" "TestPoint:TestPoint_Pad_D1.0mm"
+		(property "Footprint" "tnu:TestPoint_PinHeader_1x01_P2.54mm"
 			(at 204.47 82.55 0)
 			(hide yes)
@@
 			)
 		)
-		(property "Footprint" "TestPoint:TestPoint_Pad_D1.0mm"
+		(property "Footprint" "tnu:TestPoint_PinHeader_1x01_P2.54mm"
 			(at 204.47 64.77 0)
 			(hide yes)
@@
 			)
 		)
-		(property "Footprint" "TestPoint:TestPoint_Pad_D1.0mm"
+		(property "Footprint" "tnu:TestPoint_PinHeader_1x01_P2.54mm"
 			(at 204.47 67.31 0)
 			(hide yes)
@@
 			)
 		)
-		(property "Footprint" "TestPoint:TestPoint_Pad_D1.0mm"
+		(property "Footprint" "tnu:TestPoint_PinHeader_1x01_P2.54mm"
 			(at 204.47 90.17 0)
 			(hide yes)
